File: canbuz-1977-vw-bus-ecu.kicad_pcb (KiCad board)
At the start: 2 copper layers, 64.8 x 123.8 mm, 80 parts, among them J1 canbuz_module, J2 Conn_02x40_Counter_Clockwise, Q1 Q_NMOS_GSD, Q2 Si4497DY 36A, Q3 Q_NMOS_GSD, Q4 Si4497DY 36A, U1 open_spark_fpga, U2 VN7003ALHTR, U3 VN7003ALHTR, U4 VN7003ALHTR

Commit message: rev 08/30/2023
Parts:
- R22, R24: value 100 -> 100Ω
- R23, R25: value 10k -> 10kΩ
- R28, R31, R34: value 1k -> 1kΩ
- moved C4 34.2 mm to (70.5, 92.7)
- moved D4 34.2 mm to (63.5, 92.7)
- moved R10 34.2 mm to (68.6, 92.7)
- moved R7 34.2 mm to (72.4, 92.7)
- moved C8 34.2 mm to (66.7, 92.7)
- moved D8 32.7 mm to (61.6, 87.6)
- moved C15 32.7 mm to (68.6, 87.6)
- moved C17 32.7 mm to (64.8, 87.6)
- moved R17 32.7 mm to (72.4, 87.6)
- moved R19 32.7 mm to (70.5, 87.6)
- moved R21 32.7 mm to (66.7, 87.6)
- moved C13 25.5 mm to (69.2, 76.2), turned to 0 degrees
- moved R15 24.4 mm to (69.2, 78.1), turned to 180 degrees
- moved C11 23.6 mm to (69.2, 80.0), turned to 0 degrees
- moved D7 23.1 mm to (48.3, 69.2), turned to -90 degrees
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Connections:
- J1 pad 1: INJ5_EN -> unconnected-(J1-Pad1)
- J1 pad 12: MAP_ANALOG -> ~{FPGA_CS}
- J1 pad 13: HEAD_TEMP_ANALOG -> SCK
- J1 pad 14: OIL_PRESSURE_ANALOG -> MISO
- J1 pad 15: TPS_ANALOG -> MOSI
- J1 pad 16: O2_ANALOG -> O2_EN
- J1 pad 17: FUEL_LEVEL_ANALOG -> FPGA_EN
- J1 pad 2: 12V_ANALOG -> unconnected-(J1-Pad2)
- J1 pad 22: unconnected-(J1-Pad22) -> FUEL_PUMP_EN
- J1 pad 23: unconnected-(J1-Pad23) -> EGR_EN
- J1 pad 25: unconnected-(J1-Pad25) -> 12V_ANALOG
- J1 pad 26: unconnected-(J1-Pad26) -> FUEL_PRESSURE_ANALOG
- J1 pad 27: unconnected-(J1-Pad27) -> INTAKE_AIR_TEMP_ANALOG
- J1 pad 3: INTAKE_AIR_TEMP_ANALOG -> unconnected-(J1-Pad3)
- J1 pad 31: unconnected-(J1-Pad31) -> OIL_PRESSURE_ANALOG
- J1 pad 32: ~{FPGA_CS} -> TPS_ANALOG
- J1 pad 33: SCK -> O2_ANALOG
- J1 pad 34: MISO -> HEAD_TEMP_ANALOG
- J1 pad 35: MOSI -> MAP_ANALOG
- J1 pad 36: FUEL_PUMP_EN -> FUEL_LEVEL_ANALOG
- J1 pad 37: O2_EN -> INJ5_EN
- J1 pad 38: EGR_EN -> STARTER_EN
- J1 pad 39: FPGA_EN -> unconnected-(J1-Pad39)
- J1 pad 40: STARTER_EN -> unconnected-(J1-Pad40)
- J1 pad 5: FUEL_PRESSURE_ANALOG -> unconnected-(J1-Pad5)
Routing:
- net GND: track 175.2 -> 124.4 mm, vias 22 -> 78
- net INTAKE_AIR_TEMP: track 44.6 -> 6.30 mm
- net FUEL_PRESSURE: track 35.9 -> 2.74 mm
- net +3V3: track 104.7 -> 134.7 mm, vias 10 -> 11
- net STARTER_EN: track 28.6 -> 51.5 mm, vias 1 -> 3
- net INTAKE_AIR_TEMP_ANALOG: track 9.90 -> 30.9 mm, vias 0 -> 2
- net INJ5_EN: track 4.06 -> 24.7 mm, vias 0 -> 1
- net O2_EN: track 29.7 -> 49.5 mm, vias 0 -> 2
- net ~{FPGA_CS}: track 38.7 -> 54.2 mm
- net FUEL_PRESSURE_ANALOG: track 9.89 -> 24.7 mm, vias 0 -> 2
- net CANL: track 23.3 -> 9.94 mm
- net VBAT: track 191.2 -> 179.8 mm
- net SCK: track 42.8 -> 53.8 mm
- net FUEL_LEVEL: track 34.5 -> 45.4 mm, vias 0 -> 1
- net CANH: track 21.5 -> 13.7 mm
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Other:
- board text added: "CANBUZ 1977 VW Bus ECU Cedric Priscal 8/30/2023"
