File: canbuz-1977-vw-bus-ecu.kicad_sch (KiCad schematic)
At the start: 68 parts, among them J1 canbuz_module, J2 Conn_02x40_Counter_Clockwise, Q1 Q_NMOS_GSD, Q2 Si4497DY 36A, Q3 Q_NMOS_GSD, Q4 Si4497DY 36A, U1 open_spark_fpga

Commit message: Rev 1.0
Other:
- note removed: "TODO add ground for FUEL_LEVEL"
Changed lines of the file:
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@@
-    (effects (font (size 1.27 1.27)) (justify left bottom))
-  )
-  (text "TODO add ground for FUEL_LEVEL" (at 87.63 55.88 0)
     (effects (font (size 1.27 1.27)) (justify left bottom))
   )

Commit message: rev 08/30/2023
Parts:
- C1, C10, C11, C14, C15, C2, C3, C4, C5: Part (none) -> KAF21BR71H104KT
- C12, C13, C16, C17, C6, C7, C8, C9: Part (none) -> CGA4J2X7R1H224K125AA
- D1, D2, D3, D4, D5, D6, D7, D8: Part (none) -> NUP1301,215
- D10, D11, D12, D9: DigiKey B140-13-F -> (none); Part (none) -> B340A-13-F
- PS1: Part (none) -> TSR 2-2450
- Q1, Q3: Part (none) -> SI2302A-TP
- Q2, Q4: Part (none) -> SI4497DY-T1-GE3
- R1, R16, R17: DigiKey RC0805FR-072K2L -> (none); Part (none) -> ERJ-3GEYJ222V
- R10, R11, R14, R15, R20, R21, R5, R8: DigiKey 311-470ARCT-ND -> (none); Part (none) -> RC0603JR-07470RL
- R12: DigiKey P3.9KDACT-ND -> (none); Part (none) -> RC0603FR-073K9L
- R13: DigiKey RMCF0805FT1K00CT-ND -> (none); Part (none) -> RC0603FR-071KL
- R18, R19, R4: DigiKey 311-4.70KCRCT-ND -> (none); Part (none) -> RC0603FR-074K7L
- R2, R7: DigiKey P2.49KDACT-ND -> (none); Part (none) -> RK73H1JTTD2491F
- R22, R24: value 100 -> 100Ω; Part (none) -> RC0603FR-07100RL
- R23, R25: value 10k -> 10kΩ; Part (none) -> RC0603FR-0710KL
- R6: DigiKey P19.6KCCT-ND‎ -> (none); Part (none) -> RC0603FR-0719K6L
- R9: DigiKey 311-38.3KCRCT-ND‎ -> (none); Part (none) -> RC0603FR-0738K3L
Connections:
- net 12V_ANALOG: now also J1.25 (PA0); no longer J1.2 (PB13)
- net EGR_EN: now also J1.23 (PC15); no longer J1.38 (PB2)
- net FPGA_EN: now also J1.17 (PB7); no longer J1.39 (PB10)
- net FUEL_LEVEL_ANALOG: now also J1.36 (PB0); no longer J1.17 (PB7)
- net FUEL_PRESSURE_ANALOG: now also J1.26 (PA1); no longer J1.5 (PA8)
- net FUEL_PUMP_EN: now also J1.22 (PC14); no longer J1.36 (PB0)
- net HEAD_TEMP_ANALOG: now also J1.34 (PA6); no longer J1.13 (PB3)
- net INJ5_EN: now also J1.37 (PB1); no longer J1.1 (PB12)
- net INTAKE_AIR_TEMP_ANALOG: now also J1.27 (PA2); no longer J1.3 (PB14)
- net MAP_ANALOG: now also J1.35 (PA7); no longer J1.12 (PA15)
- net MISO: now also J1.14 (PB4); no longer J1.34 (PA6)
- net MOSI: now also J1.15 (PB5); no longer J1.35 (PA7)
- net O2_ANALOG: now also J1.33 (PA5); no longer J1.16 (PB6)
- net O2_EN: now also J1.16 (PB6); no longer J1.37 (PB1)
- net OIL_PRESSURE_ANALOG: now also J1.31 (PA3); no longer J1.14 (PB4)
- net SCK: now also J1.13 (PB3); no longer J1.33 (PA5)
- net STARTER_EN: now also J1.38 (PB2); no longer J1.40 (PB11)
- net TPS_ANALOG: now also J1.32 (PA4); no longer J1.15 (PB5)
- net ~{FPGA_CS}: now also J1.12 (PA15); no longer J1.32 (PA4)
