File: high_side_VN7003ALHTR.kicad_sch (KiCad schematic)
At the start: 4 parts, among them U2 VN7003ALHTR

Commit message: rev 08/30/2023
Parts:
- R26, R27: Part (none) -> RC0603FR-0710KL
- R28: value 1k -> 1kΩ; Part (none) -> RC0603FR-071KL
- U2: Part (none) -> VN7003AHTR
Changed lines of the file:
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@@
+      (effects (font (size 1.27 1.27)) hide)
+    )
+    (property "Part" "VN7003AHTR" (id 5) (at 152.4 95.25 0)
       (effects (font (size 1.27 1.27)) hide)
     )
@@
     )
     (property "Datasheet" "~" (id 3) (at 119.38 83.82 0)
+      (effects (font (size 1.27 1.27)) hide)
+    )
+    (property "Part" "RC0603FR-0710KL" (id 4) (at 119.38 83.82 0)
       (effects (font (size 1.27 1.27)) hide)
     )
@@
       (effects (font (size 1.27 1.27)) (justify right))
     )
-    (property "Value" "1k" (id 1) (at 132.5372 109.093 0)
+    (property "Value" "1kΩ" (id 1) (at 132.5372 109.093 0)
       (effects (font (size 1.27 1.27)) (justify right))
     )
@@
     )
     (property "Datasheet" "~" (id 3) (at 130.81 107.95 0)
+      (effects (font (size 1.27 1.27)) hide)
+    )
+    (property "Part" "RC0603FR-071KL" (id 4) (at 130.81 107.95 0)
       (effects (font (size 1.27 1.27)) hide)
     )
@@
       (effects (font (size 1.27 1.27)) hide)
     )
+    (property "Part" "RC0603FR-0710KL" (id 4) (at 110.49 88.9 0)
+      (effects (font (size 1.27 1.27)) hide)
+    )
